File: source/macrobad.kicad_pcb (KiCad board)
At the start: 2 copper layers, 98.8 x 60 mm, 11 parts, among them J1 Conn_01x04_Pin, SW1 SW_Push, SW2 SW_Push, SW3 SW_Push, SW4 SW_Push, SW5 SW_Push, SW6 RotaryEncoder_Switch, U2 MOUDLE-SEEEDUINO-XIAO

Commit message: PCB re-adjusting
Parts:
- moved D1 37.8 mm to (239.0, 130.0), turned to 180 degrees
- moved SW6 5.00 mm to (204.2, 96.5)
- moved J1 4.00 mm to (261.4, 104.9)
- moved G*** 2.86 mm to (193.4, 126.9)
Routing:
- net LED: track 35.3 -> 70.0 mm
- net VCC: track 54.7 -> 84.9 mm
